Commit message: error in load urdf

File: src/workcell_support/urdf/workcell.urdf.xacro (robot description, xacro)
@@ -27,5 +27,5 @@
 </joint>
 <!--<link name ="ur_robotiq_link"/>-->
-<!-- <joint name = "ur_to_gripper" type="fixed">
+<!-- <joint name = "ur_to_gripper" type="fixed">sss
   <parent link=""/>
   <child link="camera_frame"/>
@@ -49,3 +49,7 @@
     <origin xyz="0 0 0.025" rpy="0 0 0"/>
   </xacro:ur_robot>
+      <!--Kinect-->
+    <!-- position of kinect has to be changed in common_sensors/urdf/sensors/kinect_properties.urdf.xacro-->
+    <!--xacro:include filename="$(find common_sensors)/urdf/sensors/kinect.urdf.xacro" />
+    <xacro:sensor_kinect parent="world"/-->
 </robot>
