Commit message: Added dynamic obstacles

File: src/workcell_moveit_config/config/myworkcell.ros2_control.xacro (robot description, xacro)
@@ -50,11 +50,4 @@
                 <state_interface name="velocity"/>
             </joint>
-            <joint name="robotiq_85_left_knuckle_joint">
-                <command_interface name="position"/>
-                <state_interface name="position">
-                  <param name="initial_value">${initial_positions['robotiq_85_left_knuckle_joint']}</param>
-                </state_interface>
-                <state_interface name="velocity"/>
-            </joint>
         </ros2_control>
     </xacro:macro>

File: src/workcell_support/urdf/workcell.urdf.xacro (robot description, xacro)
@@ -15,5 +15,16 @@
   </collision>
 </link>
-<link name="camera_frame"/>
+<link name="camera_holder">
+  <visual>
+    <geometry>
+      <box size="0.01 0.01 0.5"/>
+    </geometry>
+  </visual>
+  <collision>
+    <geometry>
+      <box size="0.01 0.01 0.5"/>
+    </geometry>
+  </collision>
+</link>
 <joint name="world_to_table" type="fixed">
   <parent link="world"/>
@@ -21,11 +32,17 @@
   <origin xyz="0 0 0.5" rpy="0 0 0"/>
 </joint>
-<joint name="world_to_camera" type="fixed">
-  <parent link="world"/>
+<joint name="table_to_camera_holder" type="fixed">
+  <parent link="table"/>
+  <child link="camera_holder"/>
+  <origin xyz="-0.0 -0.250 0.25" rpy="0 0 0"/>
+</joint>
+<link name = "camera_frame"/>
+<joint name="camera_holder_to_camera_frame" type="fixed">
+  <parent link="camera_holder"/>
   <child link="camera_frame"/>
-  <origin xyz="-0.25 -0.5 1.25" rpy="0 3.14159 0"/>
+  <origin xyz="0 0 0.25" rpy="0 0 0"/>
 </joint>
 <!--<link name ="ur_robotiq_link"/>-->
-<!-- <joint name = "ur_to_gripper" type="fixed">sss
+<!-- <joint name = "ur_to_gripper" type="fixed">
   <parent link=""/>
   <child link="camera_frame"/>
@@ -53,3 +70,9 @@
     <!--xacro:include filename="$(find common_sensors)/urdf/sensors/kinect.urdf.xacro" />
     <xacro:sensor_kinect parent="world"/-->
+    <!--realsense-->
+      <xacro:arg name="use_nominal_extrinsics" default="false" />
+      <xacro:include filename="$(find realsense2_description)/urdf/_d435i.urdf.xacro"/>
+      <xacro:sensor_d435i parent="camera_frame" use_nominal_extrinsics="$(arg use_nominal_extrinsics)">
+        <origin xyz="0 0 0" rpy="0 0 0"/>
+      </xacro:sensor_d435i>
 </robot>
